File: tuner.kicad_sch (KiCad schematic)
At the start: 6 parts

Commit message: Added components
Connections:
- no-connect marks 0 -> 3
Changed lines of the file:
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@@
 		(color 0 0 0 0)
+	)
+	(no_connect
+		(at 138.43 80.01)
+	)
+	(no_connect
+		(at 138.43 96.52)
+	)
+	(no_connect
+		(at 138.43 66.04)
 	)
 	(wire
