File: voltage_regulator.kicad_sch (KiCad schematic)
At the start: 0 parts

Commit message: Added connections
Changed lines of the file:
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@@
 	(generator_version "8.0")
 	(paper "A4")
+	(text_box "There are more than one Voltage Regulator to keep one from overheating when dealing with massive currents."
+		(exclude_from_sim no)
+		(at 204.47 30.48 0)
+		(size 27.94 27.94)
+		(stroke
+			(width 0)
+			(type default)
+		)
+		(fill
+			(type none)
+		)
+		(effects
+			(font
+				(size 1.27 1.27)
+			)
+			(justify left top)
+		)
+	)
 	(hierarchical_label "GND"
 		(shape output)

Commit message: Added Probably Voltage Regulator Parts
Changed lines of the file:
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@@
+		)
+	)
+	(text_box "Might use the\n MAX1726\nhttps://www.digikey.com/en/products/detail/analog-devices-inc-maxim-integrated/MAX1725EUK-T/1517783\nhttps://www.analog.com/media/en/technical-documentation/data-sheets/max1725-max1726.pdf"
+		(exclude_from_sim no)
+		(at 88.9 71.12 0)
+		(size 118.11 39.37)
+		(stroke
+			(width 0)
+			(type default)
+		)
+		(fill
+			(type none)
+		)
+		(effects
+			(font
+				(size 1.27 1.27)
+			)
+			(justify left top)
 		)
 	)

Commit message: Added components
Parts:
- added C1, C2, C3, C4, C5: C, symbol Device:C
- added L1: L, symbol Device:L
- added R10, R11, R9: R, symbol Device:R
- added U1: ~, symbol ArmLEDLib:RT6254BHGJ6F
Connections:
- net GND: now also C1.2, C4.2, C5.2, R11.1, U1.3 (GND)
- net In: now also C1.1, U1.4 (VIN)
- net Out: now also C3.1, C4.1, C5.1, L1.2, R10.1
- new net: C2.1, U1.6 (BOOT)
- new net: C2.2, L1.1, U1.5 (LX)
- new net: C3.2, R10.2, R11.2, R9.2
- new net: R9.1, U1.1 (FB)
- new net Enable: U1.2 (EN)

Commit message: Added parts
Parts:
- C1, C4, C5: footprint (none) -> Capacitor_SMD:C_0805_2012Metric_Pad1.18x1.45mm_HandSolder
- C2: footprint (none) -> Capacitor_SMD:C_0201_0603Metric_Pad0.64x0.40mm_HandSolder
- U1: footprint (none) -> ArmLEDFootprintLib:RT6254A
Changed lines of the file:
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@@
 		)
 	)
-	(text_box "https://www.digikey.com/en/products/detail/richtek-usa-inc/RT6254BHGJ6F/6238427"
+	(text_box "https://www.digikey.com/en/products/detail/richtek-usa-inc/RT6254BHGJ6F/6238427\n\nC5, 4: https://www.digikey.com/en/products/detail/samsung-electro-mechanics/CL21A226KQCLRNC/5961171"
 		(exclude_from_sim no)
 		(at 38.1 33.02 0)
-		(size 87.63 3.81)
+		(size 87.63 21.59)
 		(stroke
 			(width 0)
@@
 			)
 		)
-		(property "Footprint" ""
+		(property "Footprint" "Capacitor_SMD:C_0201_0603Metric_Pad0.64x0.40mm_HandSolder"
 			(at 138.1252 77.47 0)
 			(effects
@@
 			)
 		)
-		(property "Datasheet" "~"
+		(property "Datasheet" "https://www.digikey.com/en/products/detail/samsung-electro-mechanics/CL10B104KO8NNNC/3886663"
 			(at 137.16 73.66 0)
 			(effects
@@
 			)
 		)
-		(property "Footprint" ""
+		(property "Footprint" "Capacitor_SMD:C_0805_2012Metric_Pad1.18x1.45mm_HandSolder"
 			(at 92.4052 77.47 0)
 			(effects
@@
 			)
 		)
-		(property "Datasheet" "~"
+		(property "Datasheet" "https://www.digikey.com/en/products/detail/tdk-corporation/C2012X5R1V226M125AC/3951664"
 			(at 91.44 73.66 0)
 			(effects
@@
 			)
 		)
-		(property "Footprint" ""
+		(property "Footprint" "Capacitor_SMD:C_0805_2012Metric_Pad1.18x1.45mm_HandSolder"
 			(at 178.7652 85.09 0)
 			(effects
@@
 			)
 		)
-		(property "Datasheet" "~"
+		(property "Datasheet" "https://www.digikey.com/en/products/detail/samsung-electro-mechanics/CL21A226KQCLRNC/5961171"
 			(at 177.8 81.28 0)
 			(effects
@@
 			)
 		)
-		(property "Footprint" ""
+		(property "Footprint" "ArmLEDFootprintLib:RT6254A"
 			(at 123.19 67.31 0)
 			(effects
@@
 			)
 		)
-		(property "Datasheet" ""
+		(property "Datasheet" "https://www.digikey.com/en/products/detail/richtek-usa-inc/RT6254BHGJ6F/6238427"
 			(at 123.19 67.31 0)
 			(effects
@@
 		(on_board yes)
 		(dnp no)
-		(fields_autoplaced yes)
 		(property "Reference" "C5"
 			(at 191.77 80.0099 0)
@@
 			)
 		)
-		(property "Footprint" ""
-			(at 188.9252 85.09 0)
-			(effects
-				(font
-					(size 1.27 1.27)
-				)
-				(hide yes)
-			)
-		)
-		(property "Datasheet" "~"
+		(property "Footprint" "Capacitor_SMD:C_0805_2012Metric_Pad1.18x1.45mm_HandSolder"
+			(at 207.01 93.726 0)
+			(effects
+				(font
+					(size 1.27 1.27)
+				)
+				(hide yes)
+			)
+		)
+		(property "Datasheet" "https://www.digikey.com/en/products/detail/samsung-electro-mechanics/CL21A226KQCLRNC/5961171"
 			(at 187.96 81.28 0)
 			(effects

Commit message: Added resistor parts + inductor
Parts:
- C3: footprint (none) -> Capacitor_SMD:C_0805_2012Metric_Pad1.18x1.45mm_HandSolder
- L1: footprint (none) -> ArmLEDFootprintLib:Inductor
- R10, R11, R9: footprint (none) -> Resistor_SMD:R_0402_1005Metric_Pad0.72x0.64mm_HandSolder
Changed lines of the file:
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@@
 		)
 	)
-	(text_box "R10: 147k ohms\nR11: 20k ohms\nL1: 4.7 micro Henries\nC1, 4, 5: 22 micro farads\nC2: 0.1 micro Farads\nC3: 47-82 pico Farads"
+	(text_box "R10: 147k ohms\nR11: 20k ohms\nR9: 5k ohms\nL1: 4.7 micro Henries\nC1, 4, 5: 22 micro farads\nC2: 0.1 micro Farads\nC3: 47-82 pico Farads"
 		(exclude_from_sim no)
 		(at 149.86 29.21 0)
@@
 			)
 		)
-		(property "Footprint" ""
+		(property "Footprint" "Resistor_SMD:R_0402_1005Metric_Pad0.72x0.64mm_HandSolder"
 			(at 156.718 88.9 90)
 			(effects
@@
 			)
 		)
-		(property "Datasheet" "~"
+		(property "Datasheet" "https://www.digikey.com/en/products/detail/vishay-dale-thin-film/PNM0402E5001BST1/4341869"
 			(at 154.94 88.9 0)
 			(effects
@@
 			)
 		)
-		(property "Footprint" ""
+		(property "Footprint" "Capacitor_SMD:C_0805_2012Metric_Pad1.18x1.45mm_HandSolder"
 			(at 166.0652 85.09 0)
 			(effects
@@
 			)
 		)
-		(property "Datasheet" "~"
+		(property "Datasheet" "https://www.digikey.com/en/products/detail/kyocera-avx/08055A640FAT2A/1602709"
 			(at 165.1 81.28 0)
 			(effects
@@
 			)
 		)
-		(property "Footprint" ""
+		(property "Footprint" "ArmLEDFootprintLib:Inductor"
 			(at 148.59 77.47 0)
 			(effects
@@
 			)
 		)
-		(property "Datasheet" "~"
+		(property "Datasheet" "https://www.digikey.com/en/products/detail/pulse-electronics/BFSI001211094R7M05/16510826"
 			(at 148.59 77.47 0)
 			(effects
@@
 			)
 		)
-		(property "Footprint" ""
+		(property "Footprint" "Resistor_SMD:R_0402_1005Metric_Pad0.72x0.64mm_HandSolder"
 			(at 142.24 86.868 90)
 			(effects
@@
 			)
 		)
-		(property "Datasheet" "~"
+		(property "Datasheet" "https://www.digikey.com/en/products/detail/vishay-dale-thin-film/PNM0402E5001BST1/4341869"
 			(at 142.24 85.09 0)
 			(effects
@@
 			)
 		)
-		(property "Footprint" ""
+		(property "Footprint" "Resistor_SMD:R_0402_1005Metric_Pad0.72x0.64mm_HandSolder"
 			(at 153.162 81.28 90)
 			(effects
@@
 			)
 		)
-		(property "Datasheet" "~"
+		(property "Datasheet" "https://www.digikey.com/en/products/detail/vishay-dale-thin-film/PNM0402E5001BST1/4341869"
 			(at 154.94 81.28 0)
 			(effects
