File: voltage_regulator.kicad_sch (KiCad schematic)
At the start: 10 parts

Commit message: Making PCB
Parts:
- removed C5: C, Capacitor_SMD:C_0805_2012Metric_Pad1.18x1.45mm_HandSolder, symbol Device:C
- removed R11: R, Resistor_SMD:R_0402_1005Metric_Pad0.72x0.64mm_HandSolder, symbol Device:R
- C1: footprint Capacitor_SMD:C_0805_2012Metric_Pad1.18x1.45mm_HandSolder -> Capacitor_SMD:C_1812_4532Metric_Pad1.57x3.40mm_HandSolder
- L1: footprint ArmLEDFootprintLib:Inductor -> ArmLEDFootprintLib:4r7007
Connections:
- net GND: now also C3.2, R10.2
- net Out: now also R9.1; no longer R10.1
- net at U1.1 (FB): now also R10.1, R9.2; no longer R9.1

Commit message: Added information
Changed lines of the file:
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@@
 		)
 	)
-	(text_box "R10: 147k ohms\nR11: 20k ohms\nR9: 5k ohms\nL1: 4.7 micro Henries\nC1, 4, 5: 22 micro farads\nC2: 0.1 micro Farads\nC3: 47-82 pico Farads"
+	(text_box "R10: 147k ohms\nR11: 20k ohms\nR9: 5k ohms\nL1: 4.7 micro Henries\nC1: 0.28 microFarads\nC4, 5: 22 micro farads\nC2: 0.1 micro Farads\nC3: 47-82 pico Farads"
 		(exclude_from_sim no)
 		(at 149.86 29.21 0)
-		(size 29.21 15.24)
+		(size 29.21 17.78)
 		(stroke
 			(width 0)
