File: ArmLEDsPrototype.kicad_sch (KiCad schematic)
At the start: 1 part

Commit message: Added connections
Parts:
- added BT1: Battery, symbol Device:Battery
- added J1: Conn_01x05, symbol Connector_Generic:Conn_01x05
- added J2, J3, J6, J7: Conn_01x02, symbol Connector_Generic:Conn_01x02
- added J4: Conn_01x01, symbol Connector_Generic:Conn_01x01
- added J5: Conn_01x03, symbol Connector_Generic:Conn_01x03
Connections:
- net +12V: now also BT1.1 (+)
- net +5V: now also A1.30 (VIN), J3.1 (Pin_1), J5.1 (Pin_1), J6.1 (Pin_1), J7.1 (Pin_1); no longer A1.27 (+5V)
- net GND: now also BT1.2 (-), J3.2 (Pin_2), J5.3 (Pin_3), J6.2 (Pin_2), J7.2 (Pin_2)
- net at A1.1 (TX1): now also J2.2 (Pin_2)
- net LED_S: now reaches A1.13 (D10)
- net LED_S: now also J5.2 (Pin_2)
- net at A1.18 (AREF): now also J4.1 (Pin_1)
- net at A1.2 (RX1): now also J2.1 (Pin_1)
- net at A1.22 (A3): now also J1.1 (Pin_1)
- net at A1.23 (SDA/A4): now also J1.2 (Pin_2)
- net at A1.24 (SCL/A5): now also J1.3 (Pin_3)
- net at A1.25 (A6): now also J1.4 (Pin_4)
- net at A1.26 (A7): now also J1.5 (Pin_5)
Other:
- moved on the sheet: A1

Commit message: Added Probably Voltage Regulator Parts
Parts:
- added J8: Conn_01x01, symbol Connector_Generic:Conn_01x01
Connections:
- net +3.3V: now reaches A1.17 (3V3)
- net +3.3V: now also J8.1 (Pin_1)
- net +12V renamed +9V

Commit message: Added components
Other:
- sheet Voltage Regulator ports: added Enable; removed GND
Changed lines of the file:
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@@
 	(paper "A4")
+	(junction
+		(at 176.53 109.22)
+		(diameter 0)
+		(color 0 0 0 0)
+	)
 	(junction
 		(at 194.31 50.8)
@@
 	(wire
 		(pts
-			(xy 176.53 111.76) (xy 180.34 111.76)
-		)
-		(stroke
-			(width 0)
-			(type default)
-		)
-	)
-	(wire
-		(pts
-			(xy 196.85 114.3) (xy 196.85 124.46)
+			(xy 176.53 109.22) (xy 180.34 109.22)
 		)
 		(stroke
@@
 	(wire
 		(pts
-			(xy 196.85 109.22) (xy 196.85 100.33)
+			(xy 196.85 111.76) (xy 196.85 100.33)
 		)
 		(stroke
@@
 	(wire
 		(pts
-			(xy 176.53 102.87) (xy 176.53 111.76)
+			(xy 176.53 100.33) (xy 176.53 109.22)
 		)
 		(stroke
@@
 	(wire
 		(pts
-			(xy 193.04 114.3) (xy 196.85 114.3)
-		)
-		(stroke
-			(width 0)
-			(type default)
-		)
-	)
-	(wire
-		(pts
 			(xy 194.31 41.91) (xy 194.31 50.8)
 		)
@@
 	(wire
 		(pts
-			(xy 193.04 109.22) (xy 196.85 109.22)
+			(xy 176.53 109.22) (xy 176.53 114.3)
+		)
+		(stroke
+			(width 0)
+			(type default)
+		)
+	)
+	(wire
+		(pts
+			(xy 176.53 114.3) (xy 180.34 114.3)
+		)
+		(stroke
+			(width 0)
+			(type default)
+		)
+	)
+	(wire
+		(pts
+			(xy 193.04 111.76) (xy 196.85 111.76)
 		)
 		(stroke
@@
 	(symbol
 		(lib_id "power:+9V")
-		(at 176.53 102.87 0)
+		(at 176.53 100.33 0)
 		(unit 1)
 		(exclude_from_sim no)
@@
 		(fields_autoplaced yes)
 		(property "Reference" "#PWR08"
-			(at 176.53 106.68 0)
+			(at 176.53 104.14 0)
 			(effects
 				(font
@@
 		)
 		(property "Value" "+9V"
-			(at 176.53 97.79 0)
+			(at 176.53 95.25 0)
 			(effects
 				(font
@@
 		)
 		(property "Footprint" ""
-			(at 176.53 102.87 0)
+			(at 176.53 100.33 0)
 			(effects
 				(font
@@
 		)
 		(property "Datasheet" ""
-			(at 176.53 102.87 0)
+			(at 176.53 100.33 0)
 			(effects
 				(font
@@
 		)
 		(property "Description" "Power symbol creates a global label with name \"+9V\""
-			(at 176.53 102.87 0)
+			(at 176.53 100.33 0)
 			(effects
 				(font
@@
 				(path "/ff63bc24-941d-4483-9b8a-1a025ec06db8"
 					(reference "#PWR08")
-					(unit 1)
-				)
-			)
-		)
-	)
-	(symbol
-		(lib_id "power:GND")
-		(at 196.85 124.46 0)
-		(unit 1)
-		(exclude_from_sim no)
-		(in_bom yes)
-		(on_board yes)
-		(dnp no)
-		(fields_autoplaced yes)
-		(property "Reference" "#PWR04"
-			(at 196.85 130.81 0)
-			(effects
-				(font
-					(size 1.27 1.27)
-				)
-				(hide yes)
-			)
-		)
-		(property "Value" "GND"
-			(at 196.85 129.54 0)
-			(effects
-				(font
-					(size 1.27 1.27)
-				)
-			)
-		)
-		(property "Footprint" ""
-			(at 196.85 124.46 0)
-			(effects
-				(font
-					(size 1.27 1.27)
-				)
-				(hide yes)
-			)
-		)
-		(property "Datasheet" ""
-			(at 196.85 124.46 0)
-			(effects
-				(font
-					(size 1.27 1.27)
-				)
-				(hide yes)
-			)
-		)
-		(property "Description" "Power symbol creates a global label with name \"GND\" , ground"
-			(at 196.85 124.46 0)
-			(effects
-				(font
-					(size 1.27 1.27)
-				)
-				(hide yes)
-			)
-		)
-		(pin "1"
-		)
-		(instances
-			(project "ArmLEDsPrototype"
-				(path "/ff63bc24-941d-4483-9b8a-1a025ec06db8"
-					(reference "#PWR04")
 					(unit 1)
 				)
@@
 			)
 		)
-		(pin "GND" input
-			(at 193.04 114.3 0)
+		(pin "Out" input
+			(at 193.04 111.76 0)
 			(effects
 				(font
@@
 			)
 		)
-		(pin "Out" input
-			(at 193.04 109.22 0)
-			(effects
-				(font
-					(size 1.27 1.27)
-				)
-				(justify right)
-			)
-		)
 		(pin "In" input
-			(at 180.34 111.76 180)
-			(effects
-				(font
+			(at 180.34 109.22 180)
+			(effects
+				(font
+					(size 1.27 1.27)
+				)
+				(justify left)
+			)
+		)
+		(pin "Enable" input
+			(at 180.34 114.3 180)
+			(effects
+				(font

Commit message: Making PCB
Connections:
- net +5V: no longer A1.30 (VIN), J3.1 (Pin_1), J5.1 (Pin_1), J6.1 (Pin_1)
- new net 5V#1: A1.30 (VIN), J5.1 (Pin_1)
- new net 5V#2: J3.1 (Pin_1)
- new net 5V#3: J6.1 (Pin_1)
Other:
- added sheet Voltage Regulator1 (voltage_regulator.kicad_sch)
- added sheet Voltage Regulator2 (voltage_regulator.kicad_sch)

Commit message: Added parts
Parts:
- J3, J6: footprint (none) -> Connector_Molex:Molex_Pico-EZmate_78171-0002_1x02-1MP_P1.20mm_Vertical
- J5: footprint (none) -> Connector_Molex:Molex_Pico-EZmate_78171-0003_1x03-1MP_P1.20mm_Vertical
Changed lines of the file:
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@@
 			)
 		)
-		(property "Footprint" ""
+		(property "Footprint" "Connector_Molex:Molex_Pico-EZmate_78171-0002_1x02-1MP_P1.20mm_Vertical"
 			(at 177.8 39.37 0)
 			(effects
@@
 			)
 		)
-		(property "Datasheet" "~"
+		(property "Datasheet" "https://www.molex.com/en-us/products/part-detail/2082940030"
 			(at 177.8 39.37 0)
 			(effects
@@
 			)
 		)
-		(property "Footprint" ""
+		(property "Footprint" "Connector_Molex:Molex_Pico-EZmate_78171-0002_1x02-1MP_P1.20mm_Vertical"
 			(at 199.39 39.37 0)
 			(effects
@@
 			)
 		)
-		(property "Datasheet" "~"
+		(property "Datasheet" "https://www.molex.com/en-us/products/part-detail/2082940030"
 			(at 199.39 39.37 0)
 			(effects
@@
 			)
 		)
-		(property "Footprint" ""
+		(property "Footprint" "Connector_Molex:Molex_Pico-EZmate_78171-0003_1x03-1MP_P1.20mm_Vertical"
 			(at 154.94 40.64 0)
 			(effects
@@
 			)
 		)
-		(property "Datasheet" "~"
+		(property "Datasheet" "https://www.molex.com/en-us/products/part-detail/2082940030"
 			(at 154.94 40.64 0)
 			(effects

Commit message: Replaced switch & pots with rotaries
Parts:
- removed J2: Conn_01x02, symbol Connector_Generic:Conn_01x02
Connections:
- net 5V#1: now also J6.1 (Pin_1); no longer A1.30 (VIN), J5.1 (Pin_1)
- net 5V#3: now also A1.30 (VIN), J5.1 (Pin_1); no longer J6.1 (Pin_1)
- net Controller/InputS: now reaches A1.2 (RX1)
- net DIPSwitches/SW1 renamed Controller/Input1B
- net DIPSwitches/SW2 renamed Controller/Input1A
- net DIPSwitches/SW3 renamed Controller/Input2B
- net DIPSwitches/SW4 renamed Controller/Input2A
- net DIPSwitches/SW5 renamed Controller/Input3B
- net DIPSwitches/SW6 renamed Controller/Input3A
- net DIPSwitches/SW7 renamed Controller/Input4B
- net DIPSwitches/SW8 renamed Controller/Input4A
- net Tuner/Out1: no longer names the net of A1.19 (A0)
- net Tuner/Out2: no longer names the net of A1.20 (A1)
- net Tuner/Out3: no longer names the net of A1.21 (A2)
Other:
- removed sheet DIPSwitches
- removed sheet Tuner
- added sheet Controller (controller.kicad_sch)

Commit message: Added information
Parts:
- removed J1: Conn_01x05, symbol Connector_Generic:Conn_01x05
- added J1: Conn_01x08, ArmLEDFootprintLib:8Pad, symbol Connector_Generic:Conn_01x08
Connections:
- net at A1.22 (A3): now also J1.4 (Pin_4)
- net at A1.23 (SDA/A4): now also J1.5 (Pin_5)
- net at A1.24 (SCL/A5): now also J1.6 (Pin_6)
- net at A1.25 (A6): now also J1.7 (Pin_7)
- net at A1.26 (A7): now also J1.8 (Pin_8)
- net at A1.19 (A0): now also J1.1 (Pin_1)
- net at A1.20 (A1): now also J1.2 (Pin_2)
- net at A1.21 (A2): now also J1.3 (Pin_3)
Changed lines of the file:
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@@
+	(wire
+		(pts
+			(xy 82.55 62.23) (xy 88.9 62.23)
+		)
+		(stroke
+			(width 0)
+			(type default)
+		)
+	)
 	(wire
 		(pts
@@
 	(wire
 		(pts
+			(xy 82.55 57.15) (xy 88.9 57.15)
+		)
+		(stroke
+			(width 0)
+			(type default)
+		)
+	)
+	(wire
+		(pts
+			(xy 82.55 59.69) (xy 88.9 59.69)
+		)
+		(stroke
+			(width 0)
+			(type default)
+		)
+	)
+	(wire
+		(pts
 			(xy 82.55 69.85) (xy 88.9 69.85)
 		)
@@
 	)
 	(symbol
-		(lib_id "Connector_Generic:Conn_01x05")
-		(at 93.98 69.85 0)
-		(unit 1)
-		(exclude_from_sim no)
-		(in_bom yes)
-		(on_board yes)
-		(dnp no)
-		(fields_autoplaced yes)
-		(property "Reference" "J1"
-			(at 96.52 68.5799 0)
-			(effects
-				(font
-					(size 1.27 1.27)
-				)
-				(justify left)
-			)
-		)
-		(property "Value" "Conn_01x05"
-			(at 96.52 71.1199 0)
-			(effects
-				(font
-					(size 1.27 1.27)
-				)
-				(justify left)
-			)
-		)
-		(property "Footprint" ""
-			(at 93.98 69.85 0)
-			(effects
-				(font
-					(size 1.27 1.27)
-				)
-				(hide yes)
-			)
-		)
-		(property "Datasheet" "~"
-			(at 93.98 69.85 0)
-			(effects
-				(font
-					(size 1.27 1.27)
-				)
-				(hide yes)
-			)
-		)
-		(property "Description" "Generic connector, single row, 01x05, script generated (kicad-library-utils/schlib/autogen/connector/)"
-			(at 93.98 69.85 0)
-			(effects
-				(font
-					(size 1.27 1.27)
-				)
-				(hide yes)
-			)
-		)
-		(pin "5"
-		)
-		(pin "1"
-		)
-		(pin "2"
-		)
-		(pin "4"
-		)
-		(pin "3"
-		)
-		(instances
-			(project "ArmLEDsPrototype"
-				(path "/ff63bc24-941d-4483-9b8a-1a025ec06db8"
-					(reference "J1")
-					(unit 1)
-				)
-			)
-		)
-	)
-	(symbol
 		(lib_id "Device:Battery")
 		(at 55.88 140.97 0)
@@
 					(unit 1)
 				)
+			)
+		)
+	)
+	(symbol
+		(lib_id "Connector_Generic:Conn_01x08")
+		(at 93.98 64.77 0)
+		(unit 1)
+		(exclude_from_sim no)
+		(in_bom yes)
+		(on_board yes)
+		(dnp no)
+		(fields_autoplaced yes)
+		(property "Reference" "J1"
+			(at 96.52 64.7699 0)
+			(effects
+				(font
+					(size 1.27 1.27)
+				)
+				(justify left)
+			)
+		)
+		(property "Value" "Conn_01x08"
+			(at 96.52 67.3099 0)
+			(effects
+				(font
+					(size 1.27 1.27)
+				)
+				(justify left)
+			)
+		)
+		(property "Footprint" "ArmLEDFootprintLib:8Pad"
+			(at 93.98 64.77 0)
+			(effects
+				(font
+					(size 1.27 1.27)
+				)
+				(hide yes)
+			)
+		)
+		(property "Datasheet" "~"
+			(at 93.98 64.77 0)
+			(effects
+				(font
+					(size 1.27 1.27)
+				)
+				(hide yes)
+			)
+		)
+		(property "Description" "Generic connector, single row, 01x08, script generated (kicad-library-utils/schlib/autogen/connector/)"
+			(at 93.98 64.77 0)
+			(effects
+				(font
+					(size 1.27 1.27)
+				)
+				(hide yes)
+			)
+		)
+		(pin "2"
+		)
+		(pin "5"
+		)
+		(pin "8"
+		)
+		(pin "6"
+		)
+		(pin "4"
+		)
+		(pin "3"
+		)
+		(pin "7"
+		)
+		(pin "1"
+		)
+		(instances
+			(project "ArmLEDsPrototype"
+				(path "/ff63bc24-941d-4483-9b8a-1a025ec06db8"
+					(reference "J1")
+					(unit 1)
+				)
